File: pcb/tide_main.kicad_pcb (KiCad board)
At the start: 2 copper layers, 127 x 81.3 mm, 48 parts, among them J1 ESP32 J3 side, J10 MOTOR DRUM, J11 MOTOR M2, J12 MOTOR O1, J13 MOTOR K1, J14 MOTOR N2, J15 MOTOR S2, J2 ESP32 J2 side, J20 HALL YEAR, J21 HALL MOON, J22 HALL M2, J23 HALL O1, J24 HALL K1, J25 HALL N2, J26 HALL S2, J3 5V IN, J4 EXP, J5 CALENDAR, Q1 IRLIB9343, Q2 2N3904, U2 MCP23017, U3 MCP23017, U4 ULN2803A, U5 ULN2803A, U6 ULN2803A, U7 74AHCT245

Commit message: Main board rev B: ESP32-C6-LCD-1.47, third MCP23017, Freerouting
- MCU is now the Waveshare ESP32-C6-LCD-1.47 in two 1x9 sockets, USB-C at
  the left edge, nothing underneath it. Only 8 free GPIOs, so a third
  MCP23017 (0x22) drives the calendar coils (via the 74AHCT245) and reads
  the year/moon latches; the ESP32 uses GPIO18/19 (I2C), 20/23 (INT), 2 (PWM)
- Board widened to 140 x 81.3 mm; silkscreen labels follow their parts
- make_board.py routes with Freerouting 2.4.1 (headless, Java 25):
  DSN export without GND -> Freerouting -> SES import -> pours, stitching,
  DRC loop. 569 segments, 8 signal vias, KiCad DRC 0 errors/0 unconnected
- +3V3 gets its own 0.3 mm class; GND clearance 0.2 (Freerouting never
  sees GND)
- BOM, Mouser list (30 lines), pin map, wiring diagram and RESUME updated

Co-Authored-By: Claude Opus 5.5 <noreply@anthropic.com>
Parts:
- added C8: 100nF, C_Disc_D5.0mm_W2.5mm_P2.50mm, F.Cu at (101.0, 97.9)
- added R9: 10k, R_Axial_DIN0207_L6.3mm_D2.5mm_P2.54mm_Vertical, F.Cu at (112.9, 80.7)
- added U8: MCP23017, DIP-28_W7.62mm_Socket, F.Cu at (80.6, 94.6)
- J1: value ESP32 J3 side -> ESP32-C6 top row; footprint PinSocket_1x19_P2.54mm_Vertical -> PinSocket_1x09_P2.54mm_Vertical
- J2: value ESP32 J2 side -> ESP32-C6 bottom row; footprint PinSocket_1x19_P2.54mm_Vertical -> PinSocket_1x09_P2.54mm_Vertical
- moved J1 44.6 mm to (51.4, 84.5), turned to 90 degrees
- moved J2 43.9 mm to (51.4, 102.2), turned to 90 degrees
- moved R7 41.5 mm to (156.0, 93.0)
- moved RN1 38.4 mm to (118.7, 100.3), turned to 0 degrees
- moved U7 37.9 mm to (120.0, 94.6), turned to 90 degrees
- moved R6 36.2 mm to (150.5, 93.0)
- moved R5 32.0 mm to (160.0, 87.5)
- moved D2 30.7 mm to (160.0, 81.0)
- moved Q2 30.6 mm to (150.5, 87.5)
- moved Q1 30.0 mm to (150.0, 81.0)
- moved C5 23.8 mm to (146.3, 86.8)
- moved C1 18.2 mm to (146.0, 102.5)
- moved F1 14.5 mm to (160.5, 108.5)
- moved RN2 14.0 mm to (84.5, 109.0)
- moved J5 13.2 mm to (175.8, 90.0)
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Connections:
- J1 pad 1: GND -> (no net)
- J1 pad 2: CTL_M1 -> (no net)
- J1 pad 3: SCL -> (no net)
- J1 pad 5: (no net) -> INT_B
- J1 pad 6: SDA -> INT_A
- J1 pad 7: GND -> SDA
- J1 pad 8: CTL_Y4 -> SCL
- J1 pad 9: CTL_Y3 -> (no net)
- J2 pad 1: +3V3 -> ESP_5V
- J2 pad 2: (no net) -> GND
- J2 pad 3: (no net) -> +3V3
- J2 pad 5: IO34 -> IO1
- J2 pad 6: (no net) -> PWM
- J2 pad 7: HALL_YEAR -> IO3
- J2 pad 8: HALL_MOON -> (no net)
- J2 pad 9: PWM -> (no net)
- J4 pad 5: IO14 -> IO1
- J4 pad 6: IO34 -> IO3
- R3 pad 1: MCP_INT -> INT_A
- U3 pad 19: MCP_INT -> INT_A
Routing:
- net INT_B: track 0.00 -> 66.6 mm, vias 0 -> 1
- net CTL_M4: track 135.3 -> 69.3 mm, vias 4 -> 0
- net INT_A: track 0.00 -> 65.2 mm, vias 0 -> 1
- net CTL_Y1: track 113.8 -> 52.1 mm, vias 1 -> 0
- net MCP_INT: track 59.9 -> 0.00 mm, vias 2 -> 0
- net CTL_Y2: track 110.2 -> 52.5 mm, vias 0 -> 1
- net CTL_M3: track 120.7 -> 63.8 mm
- net CTL_M2: track 111.0 -> 58.2 mm, vias 1 -> 0
- net CAL_M4: track 7.24 -> 57.4 mm
- net IO1: track 0.00 -> 49.9 mm
- net PWM: track 49.5 -> 98.0 mm
- net +3V3: track 234.6 -> 283.0 mm, vias 6 -> 1
- net IO3: track 0.00 -> 48.1 mm
- net IO34: track 46.4 -> 0.00 mm, vias 1 -> 0
- net CTL_Y3: track 97.3 -> 51.1 mm
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Other:
- board size 127 x 81.3 mm -> 140 x 81.3 mm
- board text added: "0"
- board text added: "12"
- board text added: "13"
- board text added: "140 × 81.3 mm · all through-hole"
- board text added: "18"
- board text added: "19"
- board text added: "2"
- board text added: "20"
- board text added: "23"
- board text added: "3"
- board text added: "4"
- board text added: "5"
- board text added: "74AHCT245 · CALENDAR 5V"
- board text added: "9"
- board text added: "C8 100n"
- board text added: "ESP32-C6-LCD-1.47"
- board text added: "G"
- board text added: "IO1"
- board text added: "IO3"
- board text added: "MCP23017 · 0x22 · CALENDAR"
- board text added: "R9 10k"
- board text added: "RX"
- board text added: "TX"
- board text added: "U8"
- board text added: "main board · rev B · ESP32-C6"
- board text added: "nothing underneath"
- board text added: "plugs in here"
- board text removed: "127 × 81.3 mm · all through-hole"
- board text removed: "74AHCT245 · CALENDAR"
- board text removed: "ESP32-DevKitC-32E"
- board text removed: "IO14"
- board text removed: "IO34"
- board text removed: "J2 side"
- board text removed: "J3 side"
- board text removed: "main board · rev A"
- board text removed: "plugs in here · nothing underneath"
